File: Eagle/DrawingBoard/PanelPCB.brd (EAGLE design)
At the start: 44.1 x 104.1 mm, 12 parts, among them M1 RARNDT-MISCELANEOUS_FEATHERBO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

Commit message: Updated DrawingBoard eagle files for cutting/printing
Other:
- board size 44.1 x 104.1 mm -> 45 x 104.1 mm
Changed lines of the file:
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@@
 <setting verticaltext="up"/>
 </settings>
-<grid distance="50" unitdist="mil" unit="mil" style="lines" multiple="1" display="no" altdistance="25" altunitdist="mil" altunit="mil"/>
+<grid distance="50" unitdist="mil" unit="mm" style="lines" multiple="1" display="no" altdistance="25" altunitdist="mil" altunit="mil"/>
 <layers>
 <layer number="1" name="Top" color="4" fill="1" visible="yes" active="yes"/>
@@
 <layer number="49" name="Reference" color="7" fill="1" visible="no" active="yes"/>
 <layer number="50" name="dxf" color="7" fill="1" visible="no" active="yes"/>
-<layer number="51" name="tDocu" color="7" fill="1" visible="yes" active="yes"/>
-<layer number="52" name="bDocu" color="7" fill="1" visible="yes" active="yes"/>
+<layer number="51" name="tDocu" color="7" fill="1" visible="no" active="yes"/>
+<layer number="52" name="bDocu" color="7" fill="1" visible="no" active="yes"/>
 <layer number="53" name="tGND_GNDA" color="7" fill="1" visible="no" active="yes"/>
 <layer number="54" name="bGND_GNDA" color="7" fill="1" visible="no" active="yes"/>
@@
 <board>
 <plain>
-<wire x1="38.1" y1="-3.81" x2="80.95" y2="-3.81" width="0" layer="20"/>
-<wire x1="80.95" y1="-3.81" x2="79.68" y2="100.32" width="0" layer="20"/>
-<wire x1="79.68" y1="100.32" x2="36.83" y2="100.32" width="0" layer="20"/>
-<wire x1="36.83" y1="100.32" x2="38.1" y2="-3.81" width="0" layer="20"/>
+<wire x1="36.068" y1="-3.81" x2="81.026" y2="-3.81" width="0" layer="20"/>
+<wire x1="81.026" y1="-3.81" x2="81.026" y2="100.33" width="0" layer="20"/>
+<wire x1="81.026" y1="100.33" x2="36.068" y2="100.33" width="0" layer="20"/>
+<wire x1="36.068" y1="100.33" x2="36.068" y2="-3.81" width="0" layer="20"/>
 <text x="67.437" y="82.55" size="1.524" layer="51" font="vector" ratio="15" distance="70" align="center">3V3
 A2
@@
 GND
 GND</text>
-<dimension x1="79.68" y1="100.32" x2="36.83" y2="100.32" x3="58.255" y3="105.41" textsize="1.778" layer="20"/>
-<dimension x1="36.83" y1="100.32" x2="36.83" y2="19.05" x3="29.21" y3="59.685" textsize="1.778" layer="20"/>
-<dimension x1="76.1746" y1="22.5552" x2="76.1746" y2="96.8248" x3="91.44" y3="59.69" textsize="1.778" layer="20"/>
 <text x="67.437" y="59.69" size="1.524" layer="51" font="vector" ratio="15" distance="70" align="center">USB
 13
@@
 SDA
 GND</text>
-<dimension x1="40.3352" y1="22.5552" x2="76.1746" y2="22.5552" x3="58.2549" y3="10.16" textsize="1.778" layer="20"/>
-<rectangle x1="48.895" y1="-3.175" x2="69.215" y2="28.575" layer="48" rot="R90"/>
 </plain>
 <attributes>
@@
 <contactref element="SV1" pad="2"/>
 <polygon width="0.4064" layer="1">
-<vertex x="35.56" y="17.78"/>
+<vertex x="35.56" y="-5.08"/>
 <vertex x="35.56" y="101.6"/>
-<vertex x="81.28" y="101.6"/>
-<vertex x="81.28" y="17.78"/>
+<vertex x="82.55" y="101.6"/>
+<vertex x="82.55" y="-5.08"/>
 </polygon>
 <polygon width="0.4064" layer="16">
-<vertex x="34.29" y="16.51"/>
+<vertex x="34.29" y="-6.35"/>
 <vertex x="34.29" y="102.87"/>
-<vertex x="82.55" y="102.87"/>
-<vertex x="82.55" y="16.51"/>
+<vertex x="83.82" y="102.87"/>
+<vertex x="83.82" y="-6.35"/>
 </polygon>
 </signal>
